File: hardware/rev/rev.kicad_pcb (KiCad board)
At the start: 2 copper layers, 29 x 100 mm, 72 parts, among them J1 USB_B_Micro, J10 Conn_02x08_Odd_Even, J2 OUT_L, J3 OUT_R, J4 Conn_01x02, J5 IN_L, J6 IN_R, SW1 SW_SPDT, SW2 SW_SPDT, SW3 SW_SPDT, U1 AMS1117-3.3, U2 RP2040, U3 W25Q128JVS, U4 AMS1117-3.3, U5 74HC04, U6 TL072, Y1 YSX321SL 12MHz Crystal

Commit message: finish zine
Parts:
- added G***: LOGO, LOGO, B.Cu at (123.4, 24.9)
- moved C30 0.07 mm to (117.7, 106.1)
Connections:
- RV2 pad MP: (no net) -> GND
Routing:
- net GND: track 157.9 -> 162.2 mm, vias 65 -> 64
